File: Fourty40.kicad_pcb (KiCad board)
At the start: 2 copper layers, 90 parts, among them SW1 SW_SPST, U1 ProMicro

Commit message: PCB Update
Parts:
- SW1: moved to F.Cu
- moved D33 53.2 mm to (259.3, 144.7)
- moved D30 53.2 mm to (164.5, 157.4)
- moved D38 53.2 mm to (128.3, 173.7)
- moved MX16 53.2 mm to (129.0, 121.0)
- moved MX4 53.2 mm to (132.3, 102.2)
- moved MX11 53.2 mm to (287.1, 100.6)
- moved MX23 53.2 mm to (290.4, 119.4)
- moved MX35 53.2 mm to (293.7, 138.1)
- moved D1 53.2 mm to (77.3, 103.3)
- moved D13 53.2 mm to (74.0, 122.1)
- moved D14 53.2 mm to (92.7, 125.4)
- moved D17 53.2 mm to (149.4, 132.8)
- moved D19 53.2 mm to (219.3, 137.5)
- moved D2 53.2 mm to (96.0, 106.6)
- moved D28 53.2 mm to (127.8, 145.8)
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Connections:
- D1 pad 1: unconnected-(D1-K-Pad1) -> ROW0
- D10 pad 1: unconnected-(D10-K-Pad1) -> ROW1
- D13 pad 1: unconnected-(D13-K-Pad1) -> ROW2
- D14 pad 1: unconnected-(D14-K-Pad1) -> ROW3
- D15 pad 1: unconnected-(D15-K-Pad1) -> ROW2
- D16 pad 1: unconnected-(D16-K-Pad1) -> ROW3
- D17 pad 1: unconnected-(D17-K-Pad1) -> ROW2
- D18 pad 1: unconnected-(D18-K-Pad1) -> ROW3
- D19 pad 1: unconnected-(D19-K-Pad1) -> ROW2
- D2 pad 1: unconnected-(D2-K-Pad1) -> ROW1
- D20 pad 1: unconnected-(D20-K-Pad1) -> ROW3
- D21 pad 1: unconnected-(D21-K-Pad1) -> ROW2
- D22 pad 1: unconnected-(D22-K-Pad1) -> ROW3
- D25 pad 1: unconnected-(D25-K-Pad1) -> ROW4
- D26 pad 1: unconnected-(D26-K-Pad1) -> ROW5
- D27 pad 1: unconnected-(D27-K-Pad1) -> ROW4
- D28 pad 1: unconnected-(D28-K-Pad1) -> ROW5
- D29 pad 1: unconnected-(D29-K-Pad1) -> ROW4
- D3 pad 1: unconnected-(D3-K-Pad1) -> ROW0
- D30 pad 1: unconnected-(D30-K-Pad1) -> ROW5
- D31 pad 1: unconnected-(D31-K-Pad1) -> ROW4
- D32 pad 1: unconnected-(D32-K-Pad1) -> ROW5
- D33 pad 1: unconnected-(D33-K-Pad1) -> ROW4
- D34 pad 1: unconnected-(D34-K-Pad1) -> ROW5
- D37 pad 1: unconnected-(D37-K-Pad1) -> ROW6
- D38 pad 1: unconnected-(D38-K-Pad1) -> ROW7
- D39 pad 1: unconnected-(D39-K-Pad1) -> ROW6
- D4 pad 1: unconnected-(D4-K-Pad1) -> ROW1
- D4 pad 2: unconnected-(D4-A-Pad2) -> Net-(D4-A)
- D40 pad 1: unconnected-(D40-K-Pad1) -> ROW7
- D41 pad 1: unconnected-(D41-K-Pad1) -> ROW6
- D42 pad 1: unconnected-(D42-K-Pad1) -> ROW7
- D5 pad 1: unconnected-(D5-K-Pad1) -> ROW0
- D5 pad 2: unconnected-(D5-A-Pad2) -> Net-(D5-A)
- D6 pad 1: unconnected-(D6-K-Pad1) -> ROW1
- D7 pad 1: unconnected-(D7-K-Pad1) -> ROW0
- D8 pad 1: unconnected-(D8-K-Pad1) -> ROW1
- D9 pad 1: unconnected-(D9-K-Pad1) -> ROW0
- MX4 pad 1: unconnected-(MX4-Pad1) -> COL1
- MX4 pad 2: unconnected-(MX4-Pad2) -> Net-(D4-A)
- MX5 pad 2: unconnected-(MX5-Pad2) -> Net-(D5-A)
- U1 pad 17: unconnected-(U1-F4-Pad17) -> COL3
Routing:
- net ROW2: track 0.00 -> 160.6 mm
- net ROW4: track 0.00 -> 160.6 mm
- net ROW5: track 0.00 -> 160.6 mm
- net ROW3: track 0.00 -> 160.6 mm
- net ROW1: track 0.00 -> 160.6 mm
- net ROW0: track 0.00 -> 160.6 mm
- net ROW6: track 0.00 -> 100.7 mm
- net ROW7: track 0.00 -> 100.7 mm
- net Net-(SW1-B): track 0.00 -> 31.6 mm
- net GND: track 0.00 -> 29.1 mm
- net Net-(D6-A): track 0.00 -> 9.77 mm
- net Net-(D1-A): track 0.00 -> 9.77 mm
- net Net-(D3-A): track 0.00 -> 9.77 mm
- net Net-(D2-A): track 0.00 -> 9.77 mm
- net Net-(D5-A): track 0.00 -> 9.77 mm
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Other:
- board outline added: 271.1 x 106.2 mm

Commit message: PCB update
Parts:
- SW1: moved to B.Cu
- moved SW1 29.9 mm to (190.8, 102.1), turned to -90 degrees
Connections:
- U1 pad 1: unconnected-(U1-D3-TX-Pad1) -> COL0
- U1 pad 17: COL3 -> COL5
- U1 pad 18: unconnected-(U1-F5-Pad18) -> COL3
- U1 pad 19: unconnected-(U1-F6-Pad19) -> COL4
- U1 pad 2: unconnected-(U1-D2-RX-Pad2) -> COL1
- U1 pad 5: unconnected-(U1-D1-Pad5) -> COL2
- U1 pad 6: unconnected-(U1-D0-Pad6) -> ROW0
- U1 pad 7: unconnected-(U1-D4-Pad7) -> ROW1
- U1 pad 8: unconnected-(U1-C6-Pad8) -> ROW2
- U1 pad 9: unconnected-(U1-D7-Pad9) -> ROW3
Routing:
- net COL1: track 0.00 -> 210.8 mm
- net COL0: track 0.00 -> 207.9 mm
- net COL4: track 0.00 -> 205.9 mm
- net COL5: track 0.00 -> 191.3 mm
- net COL2: track 0.00 -> 187.2 mm
- net COL3: track 0.00 -> 163.5 mm
- net ROW2: track 160.6 -> 279.9 mm, vias 0 -> 2
- net ROW3: track 160.6 -> 259.2 mm
- net ROW1: track 160.6 -> 255.0 mm, vias 0 -> 2
- net ROW0: track 160.6 -> 245.7 mm, vias 0 -> 2
- net ROW5: track 160.6 -> 240.5 mm
- net ROW4: track 160.6 -> 239.6 mm, vias 0 -> 2
- net ROW6: track 100.7 -> 164.9 mm, vias 0 -> 2
- net ROW7: track 100.7 -> 163.7 mm
- net Net-(SW1-B): track 31.6 -> 8.62 mm
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Other:
- outline, holes or cut-outs redrawn
