File: Fourty40.kicad_sch (KiCad schematic)
At the start: 98 parts, among them SW1 SW_SPST, U1 ProMicro

Commit message: PCB update
Parts:
- removed D45, D46, D47, D48: D_Small, Diode_SMD:D_SOD-123, symbol Device:D_Small
- removed MX45, MX46, MX47, MX48: MX_SW_HS, marbastlib-mx:SW_MX_HS_1u, symbol marbastlib-mx:MX_SW_HS
Connections:
- net COL0: no longer MX37.1, MX38.1
- net COL1: now also MX16.1, MX28.1, MX37.1, MX38.1; no longer MX39.1, MX40.1
- net COL2: now also MX39.1, MX40.1; no longer MX41.1, MX42.1
- net COL3: now also MX41.1, MX42.1; no longer MX43.1, MX44.1
- net COL4: now also MX43.1, MX44.1
- net ROW0: now also D11.1 (K)
- net ROW1: now also D12.1 (K)
- net ROW2: now also D23.1 (K)
- net ROW3: now also D24.1 (K)
- net ROW4: now also D35.1 (K)
- net ROW5: now also D36.1 (K)
- net ROW6: now also D43.1 (K)
- net ROW7: now also D44.1 (K)
- net at D22.2 (A): now also MX22.2
- net at D28.2 (A): now also MX28.2
- net at MX9.2: now also D9.2 (A)
- net at MX35.2: now also D35.2 (A)
- net at D17.2 (A): now also MX17.2
- net at MX34.2: now also D34.2 (A)
- net at D33.2 (A): now also MX33.2
- net at MX11.2: now also D11.2 (A)
- net at D10.2 (A): now also MX10.2
- net at MX23.2: now also D23.2 (A)
- net at MX40.2: now also D40.2 (A)
- net at D36.2 (A): now also MX36.2
- net at D29.2 (A): now also MX29.2
- net at MX41.2: now also D41.2 (A)
- net at MX21.2: now also D21.2 (A)
- net at MX24.2: now also D24.2 (A)
- net at D16.2 (A): now also MX16.2
- net at D12.2 (A): now also MX12.2
Other:
- moved on the sheet: D37, D38, D39, D40, D41, D42, D43, D44, MX37, MX38, MX39, MX40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

Commit message: PCB Update
Connections:
- net COL1: now also MX4.1
- net COL3: now also U1.17 (F4)
- net ROW0: now also D1.1 (K), D3.1 (K), D5.1 (K), D7.1 (K), D9.1 (K)
- net ROW1: now also D10.1 (K), D2.1 (K), D4.1 (K), D6.1 (K), D8.1 (K)
- net ROW2: now also D13.1 (K), D15.1 (K), D17.1 (K), D19.1 (K), D21.1 (K)
- net ROW3: now also D14.1 (K), D16.1 (K), D18.1 (K), D20.1 (K), D22.1 (K)
- net ROW4: now also D25.1 (K), D27.1 (K), D29.1 (K), D31.1 (K), D33.1 (K)
- net ROW5: now also D26.1 (K), D28.1 (K), D30.1 (K), D32.1 (K), D34.1 (K)
- net ROW6: now also D37.1 (K), D39.1 (K), D41.1 (K)
- net ROW7: now also D38.1 (K), D40.1 (K), D42.1 (K)
- net at D4.2 (A): now also MX4.2
- net at MX5.2: now also D5.2 (A)

Commit message: PCB update
Connections:
- net COL0: now also U1.1 (D3-TX)
- net COL1: now also U1.2 (D2-RX)
- net COL2: now also U1.5 (D1)
- net COL3: now also U1.18 (F5); no longer U1.17 (F4)
- net COL4: now also U1.19 (F6)
- net COL5: now also U1.17 (F4)
- net ROW0: now also U1.6 (D0)
- net ROW1: now also U1.7 (D4)
- net ROW2: now also U1.8 (C6)
- net ROW3: now also U1.9 (D7)
Changed lines of the file:
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@@
+    )
+  )
+  (global_label "ROW1" (shape input) (at 31.75 101.6 180) (fields_autoplaced)
+    (effects (font (size 1.27 1.27)) (justify right))
+    (property "Intersheetrefs" "${INTERSHEET_REFS}" (at 23.5828 101.6 0)
+      (effects (font (size 1.27 1.27)) (justify right) hide)
     )
   )
@@
     )
   )
-  (global_label "COL3" (shape input) (at 57.15 96.52 0) (fields_autoplaced)
+  (global_label "COL4" (shape input) (at 57.15 101.6 0) (fields_autoplaced)
     (effects (font (size 1.27 1.27)) (justify left))
-    (property "Intersheetrefs" "${INTERSHEET_REFS}" (at 64.8939 96.52 0)
+    (property "Intersheetrefs" "${INTERSHEET_REFS}" (at 64.8939 101.6 0)
+      (effects (font (size 1.27 1.27)) (justify left) hide)
+    )
+  )
+  (global_label "COL3" (shape input) (at 57.15 99.06 0) (fields_autoplaced)
+    (effects (font (size 1.27 1.27)) (justify left))
+    (property "Intersheetrefs" "${INTERSHEET_REFS}" (at 64.8939 99.06 0)
       (effects (font (size 1.27 1.27)) (justify left) hide)
     )
@@
     (effects (font (size 1.27 1.27)) (justify right))
     (property "Intersheetrefs" "${INTERSHEET_REFS}" (at 98.5128 143.51 0)
+      (effects (font (size 1.27 1.27)) (justify right) hide)
+    )
+  )
+  (global_label "ROW3" (shape input) (at 31.75 106.68 180) (fields_autoplaced)
+    (effects (font (size 1.27 1.27)) (justify right))
+    (property "Intersheetrefs" "${INTERSHEET_REFS}" (at 23.5828 106.68 0)
+      (effects (font (size 1.27 1.27)) (justify right) hide)
+    )
+  )
+  (global_label "COL0" (shape input) (at 31.75 86.36 180) (fields_autoplaced)
+    (effects (font (size 1.27 1.27)) (justify right))
+    (property "Intersheetrefs" "${INTERSHEET_REFS}" (at 24.0061 86.36 0)
+      (effects (font (size 1.27 1.27)) (justify right) hide)
+    )
+  )
+  (global_label "COL2" (shape input) (at 31.75 96.52 180) (fields_autoplaced)
+    (effects (font (size 1.27 1.27)) (justify right))
+    (property "Intersheetrefs" "${INTERSHEET_REFS}" (at 24.0061 96.52 0)
       (effects (font (size 1.27 1.27)) (justify right) hide)
     )
@@
     )
   )
+  (global_label "ROW2" (shape input) (at 31.75 104.14 180) (fields_autoplaced)
+    (effects (font (size 1.27 1.27)) (justify right))
+    (property "Intersheetrefs" "${INTERSHEET_REFS}" (at 23.5828 104.14 0)
+      (effects (font (size 1.27 1.27)) (justify right) hide)
+    )
+  )
   (global_label "COL2" (shape input) (at 180.34 35.56 90) (fields_autoplaced)
     (effects (font (size 1.27 1.27)) (justify left))
     (property "Intersheetrefs" "${INTERSHEET_REFS}" (at 180.34 27.8161 90)
       (effects (font (size 1.27 1.27)) (justify left) hide)
+    )
+  )
+  (global_label "COL1" (shape input) (at 31.75 88.9 180) (fields_autoplaced)
+    (effects (font (size 1.27 1.27)) (justify right))
+    (property "Intersheetrefs" "${INTERSHEET_REFS}" (at 24.0061 88.9 0)
+      (effects (font (size 1.27 1.27)) (justify right) hide)
     )
   )
@@
       (effects (font (size 1.27 1.27)) (justify left) hide)
     )
+  )
+  (global_label "ROW0" (shape input) (at 31.75 99.06 180) (fields_autoplaced)
+    (effects (font (size 1.27 1.27)) (justify right))
+    (property "Intersheetrefs" "${INTERSHEET_REFS}" (at 23.5828 99.06 0)
+      (effects (font (size 1.27 1.27)) (justify right) hide)
+    )
+  )
+  (global_label "COL5" (shape input) (at 57.15 96.52 0) (fields_autoplaced)
+    (effects (font (size 1.27 1.27)) (justify left))
+    (property "Intersheetrefs" "${INTERSHEET_REFS}" (at 64.8939 96.52 0)
+      (effects (font (size 1.27 1.27)) (justify left) hide)
+    )
